File: pcb/Braille-PCB-Type-5-Vertical-Motors/Braille-PCB-Type-5-Vertical-Motors.kicad_pcb (KiCad board)
At the start: 2 copper layers, 90 x 90 mm, 142 parts, among them J101 Conn_01x02, J102 Screw_Terminal_01x02, J103 Screw_Terminal_01x02, J104 Screw_Terminal_01x02, J105 Conn_01x05, J106 Conn_01x05, J107 Conn_01x08, J108 Conn_01x05, J109 Conn_01x05, J201 Conn_01x02, J202 Conn_01x02, J203 Conn_01x02, J301 Conn_01x02, J302 Conn_01x02, J303 Conn_01x02, J401 Conn_01x02, J402 Conn_01x02, J403 Conn_01x02, J501 Conn_01x02, J502 Conn_01x02, J503 Conn_01x02, M201 MountingHole, M202 MountingHole, M203 MountingHole, M301 MountingHole, M302 MountingHole, M303 MountingHole, M401 MountingHole, M402 MountingHole, M501 MountingHole, M502 MountingHole, SW101 SW_Push, SW102 SW_Push, U101 RP2040-Zero, U102 AMS1117-3.3, U103 INA219AxD, U201 AD116, U202 AD116, U203 AD116, U301 AD116, U302 AD116, U303 AD116, U401 AD116, U402 AD116, U403 AD116, U501 AD116, U502 AD116, U503 AD116, U601 74HC595, U602 74HC595, U603 74HC595

Commit message: More revision work
Parts:
- R201, R301, R401, R501: moved to F.Cu
- moved R203 122.8 mm to (50.5, 102.5)
- moved R202 120.6 mm to (52.7, 84.5), turned to -90 degrees
- moved D203 118.6 mm to (49.7, 97.5), turned to 90 degrees
- moved D201 118.6 mm to (49.7, 89.5), turned to 90 degrees
- moved D202 115.6 mm to (52.7, 93.5), turned to 90 degrees
- moved H205 114.4 mm to (49.7, 93.5)
- moved M403 113.4 mm to (61.7, 53.0)
- moved R403 113.3 mm to (62.5, 102.5)
- moved H206 111.8 mm to (52.4, 97.5)
- moved H204 111.4 mm to (52.7, 89.5)
- moved M402 110.2 mm to (64.7, 50.0)
- moved D403 109.1 mm to (61.7, 97.5), turned to 90 degrees
- moved D401 109.1 mm to (61.7, 89.5), turned to 90 degrees
- moved R402 108.8 mm to (64.7, 84.5), turned to -90 degrees
- moved D402 106.2 mm to (64.7, 93.5), turned to 90 degrees
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- renumbered H405 to H404, H406 to H405, H407 to H406, H505 to H504, H506 to H505, H507 to H506, H404 to M401, M401 to M402, M402 to M403, H504 to M501, M501 to M502, M502 to M503
Routing:
- net GND: track 222.0 -> 58.4 mm, vias 30 -> 17
- net /Braille_Cells_and_Controls/CELL2_DOT1_A: track 105.3 -> 0.00 mm, vias 4 -> 0
- net /Braille_Cells_and_Controls/CELL2_DOT1_B: track 96.6 -> 8.51 mm, vias 3 -> 2
- net /~{SHIFT_OE}: track 86.4 -> 0.00 mm, vias 5 -> 0
- net VDC: track 122.0 -> 35.8 mm, vias 6 -> 10
- net /SHIFT_SER_IN: track 81.6 -> 0.00 mm, vias 1 -> 0
- net +5V: track 98.4 -> 34.7 mm
- net /~{SHIFT_SRCLR}: track 62.5 -> 0.00 mm, vias 4 -> 0
- net /Braille_Cells_and_Controls/CELL3_DOT1_B: track 70.9 -> 8.51 mm
- net /SHIFT_SRCK: track 58.9 -> 0.00 mm, vias 4 -> 0
- net /SHIFT_RCLK: track 52.2 -> 0.00 mm, vias 2 -> 0
- net /SHIFT_SER_OUT: track 51.4 -> 0.00 mm, vias 1 -> 0
- net /Braille_Cells_and_Controls/CELL1_DOT1_B: track 54.8 -> 8.51 mm, vias 1 -> 2
- net +3V3: track 85.3 -> 46.1 mm, vias 7 -> 1
- net /UART0_RX: track 45.7 -> 9.80 mm
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- removed copper zone on B.Cu, net +3V3
- removed copper zone on B.Cu, net GND
Other:
- board size 90 x 90 mm -> 90 x 86 mm
- board text added: "Type 5 Rev 3 2025-02-09 Vertical 0408 Motors"
- board text removed: "2.5mm Intra-Cell Pitch. 6mm Inter-Cell Pitch X. Motor Pitch X: 3mm. Motor Pitch Y: 2.64mm. Top (Red) = GND Bottom (Blue) = VDC"
- board text removed: "3 - V_IN 2 - LDO 1 - RP-3V3"
- board text removed: "5V"
- board text removed: "IN"
- board text removed: "OUT"
- board text removed: "Pick LDO Input"
- board text removed: "Pick VDC Driver"
- board text removed: "RX to MCU TX from MCU"
- board text removed: "Type 5 Rev 2 2025-01-11 Vertical 0408 Motors"
- board text removed: "V_IN"
