File: pcb/Braille-PCB-Type-5-Vertical-Motors/Braille-PCB-Type-5-Vertical-Motors.kicad_pcb (KiCad board)
At the start: 2 copper layers, 90 x 86 mm, 142 parts, among them J101 Conn_01x02, J102 Screw_Terminal_01x02, J103 Screw_Terminal_01x02, J104 Screw_Terminal_01x02, J105 Conn_01x05, J106 Conn_01x05, J107 Conn_01x08, J108 Conn_01x05, J109 Conn_01x05, J201 Conn_01x02, J202 Conn_01x02, J203 Conn_01x02, J301 Conn_01x02, J302 Conn_01x02, J303 Conn_01x02, J401 Conn_01x02, J402 Conn_01x02, J403 Conn_01x02, J501 Conn_01x02, J502 Conn_01x02, J503 Conn_01x02, M201 MountingHole, M202 MountingHole, M203 MountingHole, M301 MountingHole, M302 MountingHole, M303 MountingHole, M401 MountingHole, M402 MountingHole, M403 MountingHole, M501 MountingHole, M502 MountingHole, M503 MountingHole, SW101 SW_Push, SW102 SW_Push, U101 RP2040-Zero, U102 AMS1117-3.3, U103 INA219AxD, U201 AD116, U202 AD116, U203 AD116, U301 AD116, U302 AD116, U303 AD116, U401 AD116, U402 AD116, U403 AD116, U501 AD116, U502 AD116, U503 AD116, U601 74HC595, U602 74HC595, U603 74HC595

Commit message: Finish Rev 3
Parts:
- moved R104 47.8 mm to (94.8, 112.6), turned to 180 degrees
- moved D103 47.8 mm to (94.8, 109.4)
- moved H104 1.00 mm to (113.5, 111.0)
- moved J104 0.90 mm to (100.5, 111.6)
- moved H206 0.40 mm to (52.8, 97.5)
- moved H306 0.40 mm to (58.8, 97.5)
- moved H406 0.40 mm to (64.8, 97.5)
- moved H506 0.40 mm to (70.8, 97.5)
Routing:
- net GND: track 58.4 -> 464.2 mm, vias 17 -> 32
- net VDC: track 35.8 -> 311.9 mm, vias 10 -> 25
- net +3V3: track 46.1 -> 229.1 mm, vias 1 -> 5
- net /SHIFT_RCLK: track 0.00 -> 167.2 mm, vias 0 -> 5
- net /SHIFT_SRCK: track 0.00 -> 165.8 mm, vias 0 -> 5
- net /Braille_Cells_and_Controls/CELL2_DOT1_B: track 8.51 -> 168.7 mm, vias 2 -> 8
- net /Braille_Cells_and_Controls/CELL2_DOT1_A: track 0.00 -> 158.4 mm, vias 0 -> 7
- net /~{SHIFT_SRCLR}: track 0.00 -> 157.6 mm, vias 0 -> 6
- net /~{SHIFT_OE}: track 0.00 -> 125.4 mm, vias 0 -> 4
- net /Braille_Cells_and_Controls/CELL1_DOT3_A: track 0.00 -> 119.1 mm, vias 0 -> 2
- net /Braille_Cells_and_Controls/CELL2_DOT2_B: track 8.68 -> 127.6 mm, vias 2 -> 5
- net /SHIFT_SER_IN: track 0.00 -> 118.0 mm, vias 0 -> 2
- net /Braille_Cells_and_Controls/CELL2_DOT3_A: track 0.00 -> 105.0 mm, vias 0 -> 4
- net Net-(U601-QH'): track 0.00 -> 95.3 mm, vias 0 -> 4
- net /Braille_Cells_and_Controls/CELL3_DOT1_A: track 0.00 -> 93.1 mm, vias 0 -> 4
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Other:
- board text added: "IN/OUT"
- board text added: "No bottom pins"
- board text added: "VDC GND"
- board text removed: "V_IN GND"
