File: pcb/Braille-PCB-Type-5-Vertical-Motors/Braille_Cells_and_Controls.kicad_sch (KiCad schematic)
At the start: 6 parts, among them U26 74HC595, U27 74HC595, U28 74HC595

Commit message: PCB: Work on new revision
Parts:
- renumbered C27 to C601, C30 to C602, C31 to C603, U26 to U601, U27 to U602, U28 to U603
Changed lines of the file:
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@@
 		(on_board yes)
 		(dnp no)
-		(property "Reference" "#PWR0117"
+		(property "Reference" "#PWR0603"
 			(at 175.26 31.75 0)
 			(effects
@@
 			(project "Braille-PCB-Type-5-Vertical-Motors"
 				(path "/3829a125-89bd-48f9-bfbe-92d753eb8f7f/508cfeb6-61a5-4af4-970c-045ef9c703bd"
-					(reference "#PWR0117")
+					(reference "#PWR0603")
 					(unit 1)
 				)
@@
 		(dnp no)
 		(fields_autoplaced yes)
-		(property "Reference" "U26"
+		(property "Reference" "U601"
 			(at 55.5341 25.4 0)
 			(effects
@@
 			(project "Braille-PCB-Type-5-Vertical-Motors"
 				(path "/3829a125-89bd-48f9-bfbe-92d753eb8f7f/508cfeb6-61a5-4af4-970c-045ef9c703bd"
-					(reference "U26")
+					(reference "U601")
 					(unit 1)
 				)
@@
 		(on_board yes)
 		(dnp no)
-		(property "Reference" "#PWR0114"
+		(property "Reference" "#PWR0604"
 			(at 53.34 67.31 0)
 			(effects
@@
 			(project "Braille-PCB-Type-5-Vertical-Motors"
 				(path "/3829a125-89bd-48f9-bfbe-92d753eb8f7f/508cfeb6-61a5-4af4-970c-045ef9c703bd"
-					(reference "#PWR0114")
+					(reference "#PWR0604")
 					(unit 1)
 				)
@@
 		(on_board yes)
 		(dnp no)
-		(property "Reference" "#PWR0132"
+		(property "Reference" "#PWR0608"
 			(at 36.83 83.82 0)
 			(effects
@@
 			(project "Braille-PCB-Type-5-Vertical-Motors"
 				(path "/3829a125-89bd-48f9-bfbe-92d753eb8f7f/508cfeb6-61a5-4af4-970c-045ef9c703bd"
-					(reference "#PWR0132")
+					(reference "#PWR0608")
 					(unit 1)
 				)
@@
 		(on_board yes)
 		(dnp no)
-		(property "Reference" "#PWR0113"
+		(property "Reference" "#PWR0601"
 			(at 53.34 31.75 0)
 			(effects
@@
 			(project "Braille-PCB-Type-5-Vertical-Motors"
 				(path "/3829a125-89bd-48f9-bfbe-92d753eb8f7f/508cfeb6-61a5-4af4-970c-045ef9c703bd"
-					(reference "#PWR0113")
+					(reference "#PWR0601")
 					(unit 1)
 				)
@@
 		(dnp no)
 		(fields_autoplaced yes)
-		(property "Reference" "C27"
+		(property "Reference" "C601"
 			(at 27.94 83.8199 0)
 			(effects
@@
 			(project "Braille-PCB-Type-5-Vertical-Motors"
 				(path "/3829a125-89bd-48f9-bfbe-92d753eb8f7f/508cfeb6-61a5-4af4-970c-045ef9c703bd"
-					(reference "C27")
+					(reference "C601")
 					(unit 1)
 				)
@@
 		(on_board yes)
 		(dnp no)
-		(property "Reference" "#PWR0115"
+		(property "Reference" "#PWR0602"
 			(at 114.3 31.75 0)
 			(effects
@@
 			(project "Braille-PCB-Type-5-Vertical-Motors"
 				(path "/3829a125-89bd-48f9-bfbe-92d753eb8f7f/508cfeb6-61a5-4af4-970c-045ef9c703bd"
-					(reference "#PWR0115")
+					(reference "#PWR0602")
 					(unit 1)
 				)
@@
 		(dnp no)
 		(fields_autoplaced yes)
-		(property "Reference" "U27"
+		(property "Reference" "U602"
 			(at 116.4941 25.4 0)
 			(effects
@@
 			(project "Braille-PCB-Type-5-Vertical-Motors"
 				(path "/3829a125-89bd-48f9-bfbe-92d753eb8f7f/508cfeb6-61a5-4af4-970c-045ef9c703bd"
-					(reference "U27")
+					(reference "U602")
 					(unit 1)
 				)
@@
 		(dnp no)
 		(fields_autoplaced yes)
-		(property "Reference" "C30"
+		(property "Reference" "C602"
 			(at 40.64 83.8199 0)
 			(effects
@@
 			(project "Braille-PCB-Type-5-Vertical-Motors"
 				(path "/3829a125-89bd-48f9-bfbe-92d753eb8f7f/508cfeb6-61a5-4af4-970c-045ef9c703bd"
-					(reference "C30")
+					(reference "C602")
 					(unit 1)
 				)
@@
 		(dnp no)
 		(fields_autoplaced yes)
-		(property "Reference" "#PWR0135"
+		(property "Reference" "#PWR0611"
 			(at 36.83 96.52 0)
 			(effects
@@
 			(project "Braille-PCB-Type-5-Vertical-Motors"
 				(path "/3829a125-89bd-48f9-bfbe-92d753eb8f7f/508cfeb6-61a5-4af4-970c-045ef9c703bd"
-					(reference "#PWR0135")
+					(reference "#PWR0611")
 					(unit 1)
 				)
@@
 		(dnp no)
 		(fields_autoplaced yes)
-		(property "Reference" "#PWR0133"
+		(property "Reference" "#PWR0610"
 			(at 24.13 96.52 0)
 			(effects
@@
 			(project "Braille-PCB-Type-5-Vertical-Motors"
 				(path "/3829a125-89bd-48f9-bfbe-92d753eb8f7f/508cfeb6-61a5-4af4-970c-045ef9c703bd"
-					(reference "#PWR0133")
+					(reference "#PWR0610")
 					(unit 1)
 				)
@@
 		(on_board yes)
 		(dnp no)
-		(property "Reference" "#PWR0118"
+		(property "Reference" "#PWR0606"
 			(at 175.26 67.31 0)
 			(effects
@@
 			(project "Braille-PCB-Type-5-Vertical-Motors"
 				(path "/3829a125-89bd-48f9-bfbe-92d753eb8f7f/508cfeb6-61a5-4af4-970c-045ef9c703bd"
-					(reference "#PWR0118")
+					(reference "#PWR0606")
 					(unit 1)
 				)
@@
 		(dnp no)
 		(fields_autoplaced yes)
-		(property "Reference" "#PWR0137"
+		(property "Reference" "#PWR0612"
 			(at 49.53 96.52 0)
 			(effects
@@
 			(project "Braille-PCB-Type-5-Vertical-Motors"
 				(path "/3829a125-89bd-48f9-bfbe-92d753eb8f7f/508cfeb6-61a5-4af4-970c-045ef9c703bd"
-					(reference "#PWR0137")
+					(reference "#PWR0612")
 					(unit 1)
 				)
@@
 		(on_board yes)
 		(dnp no)
-		(property "Reference" "#PWR0136"
+		(property "Reference" "#PWR0609"
 			(at 49.53 83.82 0)
 			(effects
@@
 			(project "Braille-PCB-Type-5-Vertical-Motors"
 				(path "/3829a125-89bd-48f9-bfbe-92d753eb8f7f/508cfeb6-61a5-4af4-970c-045ef9c703bd"
-					(reference "#PWR0136")
+					(reference "#PWR0609")
 					(unit 1)
 				)
@@
 		(dnp no)
 		(fields_autoplaced yes)
-		(property "Reference" "C31"
+		(property "Reference" "C603"
 			(at 53.34 83.8199 0)
 			(effects
@@
 			(project "Braille-PCB-Type-5-Vertical-Motors"
 				(path "/3829a125-89bd-48f9-bfbe-92d753eb8f7f/508cfeb6-61a5-4af4-970c-045ef9c703bd"
-					(reference "C31")
+					(reference "C603")
 					(unit 1)
 				)
@@
 		(dnp no)
 		(fields_autoplaced yes)
-		(property "Reference" "U28"
+		(property "Reference" "U603"
 			(at 177.4541 25.4 0)
 			(effects
@@
 			(project "Braille-PCB-Type-5-Vertical-Motors"
 				(path "/3829a125-89bd-48f9-bfbe-92d753eb8f7f/508cfeb6-61a5-4af4-970c-045ef9c703bd"
-					(reference "U28")
+					(reference "U603")
 					(unit 1)
 				)
@@
 		(on_board yes)
 		(dnp no)
-		(property "Reference" "#PWR0134"
+		(property "Reference" "#PWR0607"
 			(at 24.13 83.82 0)
 			(effects
@@
 			(project "Braille-PCB-Type-5-Vertical-Motors"
 				(path "/3829a125-89bd-48f9-bfbe-92d753eb8f7f/508cfeb6-61a5-4af4-970c-045ef9c703bd"
-					(reference "#PWR0134")
+					(reference "#PWR0607")
 					(unit 1)
 				)
@@
 		(on_board yes)
 		(dnp no)
-		(property "Reference" "#PWR0116"
+		(property "Reference" "#PWR0605"
 			(at 114.3 67.31 0)
 			(effects
@@
 			(project "Braille-PCB-Type-5-Vertical-Motors"
 				(path "/3829a125-89bd-48f9-bfbe-92d753eb8f7f/508cfeb6-61a5-4af4-970c-045ef9c703bd"
-					(reference "#PWR0116")
-					(unit 1)
-				)
+					(reference "#PWR0605")
+					(unit 1)
+				)
