File: pcb/Braille-PCB-Type-5-Vertical-Motors/Braille_Cell.kicad_sch (KiCad schematic)
At the start: 21 parts, among them J10 Conn_01x02, J14 Conn_01x02, J18 Conn_01x02, M10 Motor_DC, M2 Motor_DC, M6 Motor_DC, U10 AD116, U8 AD116, U9 AD116

Commit message: PCB: Work on new revision
Parts:
- removed D10, D8, D9: LED_Dual_Bidirectional, 00-project-footprints:LED_0603_1608Metric_HandSolder_2x_Reverse, symbol Device:LED_Dual_Bidirectional
- removed M10, M2, M6: Motor_DC, 00-project-footprints:Motor_Tiny_0408_Vertical, symbol Motor:Motor_DC
- removed R21, R22: 5k1, Resistor_SMD:R_0603_1608Metric_Pad0.98x0.95mm_HandSolder, symbol Device:R
- added D201, D202, D203: LED_Dual_AAKK, 00-project-footprints:LED_1206_Bicolor_AAKK, symbol Device:LED_Dual_AAKK
- added H204, H205, H206: MountingHole, 00-project-footprints:Hole_for_Motor_Shaft, symbol Mechanical:MountingHole
- added M201, M202, M203: MountingHole, 00-project-footprints:Motor_Tiny_0408_Vertical, symbol Mechanical:MountingHole
- added R202, R203: 5k1, Resistor_SMD:R_0603_1608Metric_Pad0.98x0.95mm_HandSolder, symbol Device:R
- renumbered C8 to C301, C9 to C302, C10 to C303, H14 to H301, H18 to H302, H22 to H303, J10 to J301, J14 to J302, J18 to J303, R20 to R301, U8 to U301, U9 to U302, U10 to U303
Connections:
- net DOT1_B_CTRL: now also D201.2 (A2), D201.3 (K1)
- net DOT2_A_CTRL: now also R202.1
- net DOT2_B_CTRL: now also D202.2 (A2), D202.3 (K1)
- net DOT3_A_CTRL: now also R203.1
- net DOT3_B_CTRL: now also D203.2 (A2), D203.3 (K1)
- net at R301.2: now also D201.1 (A1), D201.4 (K2)
- new net: D203.1 (A1), D203.4 (K2), R203.2
- new net: D202.1 (A1), D202.4 (K2), R202.2
Other:
- note added: "Light guide from lower layer."

Commit message: Finish Rev 3
Parts:
- renumbered D201 to D301, D202 to D302, D203 to D303, H204 to H304, H205 to H305, H206 to H306, M201 to M301, M202 to M302, M203 to M303, R202 to R302, R203 to R303
Changed lines of the file:
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@@
 	(paper "USLetter")
 	(title_block
-		(date "2025-01-11")
-		(rev "Type 5 Rev 2")
+		(date "2025-02-08")
+		(rev "Type 5 Rev 3")
 	)
 	(junction
@@
 		(dnp no)
 		(fields_autoplaced yes)
-		(property "Reference" "H205"
+		(property "Reference" "H305"
 			(at 213.995 121.2849 0)
 			(effects
@@
 		(dnp no)
 		(fields_autoplaced yes)
-		(property "Reference" "H204"
+		(property "Reference" "H304"
 			(at 217.805 116.2049 0)
 			(effects
@@
 		(on_board yes)
 		(dnp no)
-		(property "Reference" "D203"
+		(property "Reference" "D303"
 			(at 212.09 80.264 90)
 			(effects
@@
 		(dnp no)
 		(fields_autoplaced yes)
-		(property "Reference" "R203"
+		(property "Reference" "R303"
 			(at 213.36 68.5799 0)
 			(effects
@@
 		(on_board yes)
 		(dnp no)
-		(property "Reference" "M201"
+		(property "Reference" "M301"
 			(at 146.05 83.82 0)
 			(effects
@@
 		(on_board yes)
 		(dnp no)
-		(property "Reference" "D202"
+		(property "Reference" "D302"
 			(at 237.49 58.674 90)
 			(effects
@@
 		(on_board yes)
 		(dnp no)
-		(property "Reference" "M202"
+		(property "Reference" "M302"
 			(at 175.26 116.84 0)
 			(effects
@@
 		(dnp no)
 		(fields_autoplaced yes)
-		(property "Reference" "R202"
+		(property "Reference" "R302"
 			(at 238.76 46.9899 0)
 			(effects
@@
 		(dnp no)
 		(fields_autoplaced yes)
-		(property "Reference" "H206"
+		(property "Reference" "H306"
 			(at 217.805 126.3649 0)
 			(effects
@@
 		(on_board yes)
 		(dnp no)
-		(property "Reference" "D201"
+		(property "Reference" "D301"
 			(at 212.09 35.814 90)
 			(effects
@@
 		(on_board yes)
 		(dnp no)
-		(property "Reference" "M203"
+		(property "Reference" "M303"
 			(at 149.86 151.13 0)
 			(effects

Commit message: pcb: Bump to KiCAD v9
Parts:
- renumbered C301 to C201, C302 to C202, C303 to C203, D301 to D201, D302 to D202, D303 to D203, H301 to H201, H302 to H202, H303 to H203, H304 to H204, H305 to H205, H306 to H206, J301 to J201, J302 to J202, J303 to J203, M301 to M201, M302 to M202, M303 to M203, R301 to R201, R302 to R202, R303 to R203, U301 to U201, U302 to U202, U303 to U203

Commit message: pcb: Motor driver model schematic comment
Parts:
- U201, U202, U203: value AD116 -> AD116/BDR6120S
Changed lines of the file:
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@@
 		(fields_autoplaced yes)
 		(property "Reference" "U203"
-			(at 89.8241 140.97 0)
-			(effects
-				(font
-					(size 1.27 1.27)
-				)
-				(justify left)
-			)
-		)
-		(property "Value" "AD116"
-			(at 89.8241 143.51 0)
+			(at 89.7733 140.97 0)
+			(effects
+				(font
+					(size 1.27 1.27)
+				)
+				(justify left)
+			)
+		)
+		(property "Value" "AD116/BDR6120S"
+			(at 89.7733 143.51 0)
 			(effects
 				(font
@@
 		(fields_autoplaced yes)
 		(property "Reference" "U201"
-			(at 89.8241 73.66 0)
-			(effects
-				(font
-					(size 1.27 1.27)
-				)
-				(justify left)
-			)
-		)
-		(property "Value" "AD116"
-			(at 89.8241 76.2 0)
+			(at 89.7733 73.66 0)
+			(effects
+				(font
+					(size 1.27 1.27)
+				)
+				(justify left)
+			)
+		)
+		(property "Value" "AD116/BDR6120S"
+			(at 89.7733 76.2 0)
 			(effects
 				(font
@@
 		(fields_autoplaced yes)
 		(property "Reference" "U202"
-			(at 116.4941 106.68 0)
-			(effects
-				(font
-					(size 1.27 1.27)
-				)
-				(justify left)
-			)
-		)
-		(property "Value" "AD116"
-			(at 116.4941 109.22 0)
-			(effects
-				(font
+			(at 116.4433 106.68 0)
+			(effects
+				(font
+					(size 1.27 1.27)
+				)
+				(justify left)
+			)
+		)
+		(property "Value" "AD116/BDR6120S"
+			(at 116.4433 109.22 0)
+			(effects
+				(font
